Commit message: merge in changes from scheckie/drc_ws

File: src/droid_description/urdf/droid.xacro (robot description, xacro)
@@ -9,5 +9,5 @@
     <pose>0 0 0.1 0 0 0</pose>
     <inertial>
-      <mass value="15.0"/>
+      <mass value="1.0"/>
       <origin xyz="0.0 0 0.1" rpy=" 0 0 0"/>
       <inertia
@@ -164,12 +164,12 @@
     <child link="camera"/>
   </joint>
-  <joint name="hokuyo_joint" type="fixed">
+  <!--joint name="hokuyo_joint" type="fixed">
     <axis xyz="0 1 0" />
     <origin xyz=".15 0 .1" rpy="0 0 0"/>
     <parent link="chassis"/>
     <child link="hokuyo"/>
-  </joint>
+  </joint-->
   <!-- Hokuyo Laser -->
-  <link name="hokuyo">
+  <!--link name="hokuyo">
     <collision>
       <origin xyz="0 0 0" rpy="0 0 0"/>
@@ -189,4 +189,4 @@
       <inertia ixx="1e-6" ixy="0" ixz="0" iyy="1e-6" iyz="0" izz="1e-6" />
     </inertial>
-  </link>
+  </link-->
 </robot>
